File: KiCad/Atari-PC1-XT-Adapter.sch (KiCad schematic (older format))
At the start: 3 parts, among them J1 ISA_8bit Slot, J2 Conn_2Rows-49Pins, J8 Conn_2Rows-49Pins

Commit message: Update XT-Adapter
Parts:
- added J3: Conn_01x04, Connector_PinHeader_2.54mm:PinHeader_1x04_P2.54mm_Vertical, symbol Connector_Generic:Conn_01x04
- J1: footprint (none) -> Connector_PinHeader_2.54mm:PinHeader_2x31_P2.54mm_Vertical; symbol Connector:Bus_ISA_8bit -> Atari-PC1-XT-Adapter-rescue:Bus_ISA_8bit-Connector
- J2, J8: footprint (none) -> Connector_PinHeader_2.54mm:PinHeader_2x25_P2.54mm_Vertical
Connections:
- net +12V: now also J3.1 (Pin_1)
- net +5V: now also J3.3 (Pin_3)
- net -12V: now also J3.2 (Pin_2)
- net -5V: now also J3.4 (Pin_4)
Changed lines of the file:
@@
 $EndDescr
 $Comp
-L Connector:Bus_ISA_8bit J1
+L Atari-PC1-XT-Adapter-rescue:Bus_ISA_8bit-Connector J1
 U 1 1 60F9F3FA
 P 5800 3450
 F 0 "J1" H 5800 5217 50  0001 C CNN
 F 1 "ISA_8bit Slot" H 5800 5126 50  0000 C CNB
-F 2 "" H 5800 3450 50  0001 C CNN
+F 2 "Connector_PinHeader_2.54mm:PinHeader_2x31_P2.54mm_Vertical" H 5800 3450 50  0001 C CNN
 F 3 "https://en.wikipedia.org/wiki/Industry_Standard_Architecture" H 5800 3450 50  0001 C CNN
 	1    5800 3450
@@
 F 0 "J2" H 3250 4817 50  0000 C CNB
 F 1 "Conn_2Rows-49Pins" H 3250 4726 50  0001 C CNN
-F 2 "" H 3200 3400 50  0001 C CNN
+F 2 "Connector_PinHeader_2.54mm:PinHeader_2x25_P2.54mm_Vertical" H 3200 3400 50  0001 C CNN
 F 3 "~" H 3200 3400 50  0001 C CNN
 	1    3200 3400
@@
 F 0 "J8" H 8400 4775 50  0000 C CNB
 F 1 "Conn_2Rows-49Pins" H 8400 4776 50  0001 C CNN
-F 2 "" H 8350 3450 50  0001 C CNN
+F 2 "Connector_PinHeader_2.54mm:PinHeader_2x25_P2.54mm_Vertical" H 8350 3450 50  0001 C CNN
 F 3 "~" H 8350 3450 50  0001 C CNN
 	1    8350 3450
@@
 	5100 2350 5000 2350
 Wire Wire Line
-	5000 2350 5000 1150
-Wire Wire Line
 	5100 2550 4500 2550
 Wire Wire Line
@@
 Wire Wire Line
 	5100 2750 4300 2750
-Wire Wire Line
-	4300 1050 4300 1100
 $Comp
 L power:+5V #PWR0104
@@
 Wire Wire Line
 	3400 2450 5100 2450
-Wire Wire Line
-	4700 1050 4700 1300
-Wire Wire Line
-	4500 2550 4500 1200
 NoConn ~ 5100 2650
 Wire Wire Line
@@
 Wire Wire Line
 	2450 5350 2450 5200
-$Comp
-L power:PWR_FLAG #FLG0102
-U 1 1 6100CD45
-P 4300 1100
-F 0 "#FLG0102" H 4300 1175 50  0001 C CNN
-F 1 "PWR_FLAG" V 4300 1227 50  0000 L CNN
-F 2 "" H 4300 1100 50  0001 C CNN
-F 3 "~" H 4300 1100 50  0001 C CNN
-	1    4300 1100
-	0    -1   -1   0
-$EndComp
-Connection ~ 4300 1100
-Wire Wire Line
-	4300 1100 4300 2750
-$Comp
-L power:PWR_FLAG #FLG0103
-U 1 1 61020315
-P 4500 1200
-F 0 "#FLG0103" H 4500 1275 50  0001 C CNN
-F 1 "PWR_FLAG" V 4500 1327 50  0000 L CNN
-F 2 "" H 4500 1200 50  0001 C CNN
-F 3 "~" H 4500 1200 50  0001 C CNN
-	1    4500 1200
-	0    -1   -1   0
-$EndComp
-Connection ~ 4500 1200
-Wire Wire Line
-	4500 1200 4500 1050
-$Comp
-L power:PWR_FLAG #FLG0104
-U 1 1 61020BAD
-P 4700 1300
-F 0 "#FLG0104" H 4700 1375 50  0001 C CNN
-F 1 "PWR_FLAG" V 4700 1427 50  0000 L CNN
-F 2 "" H 4700 1300 50  0001 C CNN
-F 3 "~" H 4700 1300 50  0001 C CNN
-	1    4700 1300
-	0    -1   -1   0
-$EndComp
-Connection ~ 4700 1300
-Wire Wire Line
-	4700 1300 4700 2150
-$Comp
-L power:PWR_FLAG #FLG0105
-U 1 1 61020FF3
-P 5000 1150
-F 0 "#FLG0105" H 5000 1225 50  0001 C CNN
-F 1 "PWR_FLAG" V 5000 1278 50  0000 L CNN
-F 2 "" H 5000 1150 50  0001 C CNN
-F 3 "~" H 5000 1150 50  0001 C CNN
-	1    5000 1150
-	0    1    1    0
-$EndComp
-Connection ~ 5000 1150
-Wire Wire Line
-	5000 1150 5000 1050
 NoConn ~ 3400 2200
 NoConn ~ 6500 1950
+$Comp
+L Connector_Generic:Conn_01x04 J3
+U 1 1 61219C3F
+P 5600 1150
+F 0 "J3" H 5680 1142 50  0000 L CNN
+F 1 "Conn_01x04" H 5680 1051 50  0000 L CNN
+F 2 "Connector_PinHeader_2.54mm:PinHeader_1x04_P2.54mm_Vertical" H 5600 1150 50  0001 C CNN
+F 3 "~" H 5600 1150 50  0001 C CNN
+	1    5600 1150
+	1    0    0    -1
+$EndComp
+Wire Wire Line
+	5000 1050 5000 1350
+Wire Wire Line
+	4300 1050 4300 2750
+Wire Wire Line
+	4500 1050 4500 1150
+Wire Wire Line
+	4700 1050 4700 1250
+Connection ~ 4300 1050
+Wire Wire Line
+	4500 1150 5400 1150
+Connection ~ 4500 1150
+Wire Wire Line
+	4500 1150 4500 2550
+Wire Wire Line
+	4700 1250 5400 1250
+Connection ~ 4700 1250
+Wire Wire Line
+	4700 1250 4700 2150
+Wire Wire Line
+	5000 1350 5400 1350
+Connection ~ 5000 1350
+Wire Wire Line
+	5000 1350 5000 2350
+Wire Wire Line
+	4300 1050 5400 1050
 $EndSCHEMATC

Commit message: Update PCB
Parts:
- J1: symbol Atari-PC1-XT-Adapter-rescue:Bus_ISA_8bit-Connector -> Connector:Bus_ISA_8bit
Changed lines of the file:
@@
 $EndDescr
 $Comp
-L Atari-PC1-XT-Adapter-rescue:Bus_ISA_8bit-Connector J1
+L Connector:Bus_ISA_8bit J1
 U 1 1 60F9F3FA
 P 5800 3450
 F 0 "J1" H 5800 5217 50  0001 C CNN
 F 1 "ISA_8bit Slot" H 5800 5126 50  0000 C CNB
-F 2 "Connector_PinHeader_2.54mm:PinHeader_2x31_P2.54mm_Vertical" H 5800 3450 50  0001 C CNN
+F 2 "Connector_PinHeader_2.54mm:PinHeader_2x31_P2.54mm_Vertical" H 5827 1796 50  0000 C CNN
 F 3 "https://en.wikipedia.org/wiki/Industry_Standard_Architecture" H 5800 3450 50  0001 C CNN
 	1    5800 3450
